File: KiCad/Integrated_System/integrated_system/ECU.kicad_sch (KiCad schematic)
At the start: 41 parts

Commit message: Updated Footprint v1.1
Parts:
- removed ON/OFF_SWITCH?: SW_DPDT_x2, symbol Switch:SW_DPDT_x2
- added SW1, SW2: SW_SPDT, symbol Switch:SW_SPDT
- added SW3: SW_Push, symbol Switch:SW_Push
- U4: renamed from U?; footprint (none) -> Library:Mini360
- gave numbers to parts that had none: 33
Connections:
- net +12V: now also SW1.2 (B)
- net FP_12V: now also SW1.1 (A)
- net GND: now also SW3.1
- net at A1.10 (IO4/A5): now also SW2.1 (A)
- net at A1.9 (IO36/A4): now also SW3.2
- net at D4.2 (A): now also SW1.3 (C)
- new net VDD (+ 3.3 V): SW2.2 (B)
- no-connect marks 25 -> 24

Commit message: Started PCB layout
Parts:
- removed U1: SCD30, SCD30:MODULE_SCD30, symbol SCD30:SCD30
- removed U2: SGP30, SGP30:SGP30, symbol SGP30:SGP30
- removed U3: BME680, BME680:PSON80P300X300X100-8N, symbol BME680:BME680
- added U1: SGP30, SGP30:SGP30, symbol SGP30:SGP30
- added U2: BME680, BME680:PSON80P300X300X100-8N, symbol BME680:BME680
- added U5: SCD30, SCD30:MODULE_SCD30, symbol SCD30:SCD30
Connections:
- net GND: now also U1.2 (VSS), U2.1 (GND), U2.7 (GND), U5.2 (GND)
- net VDD: now also U1.1 (VDD), U2.8 (VDD), U5.1 (VDD)
- net at A1.18 (SCL/IO22): now also U1.6 (SCL), U2.4 (SCK), U5.3 (TX/SCL)
- net at A1.17 (SDA/IO23): now also U1.3 (SDA), U2.3 (SDI), U5.4 (RX/SDA)

Commit message: Updated Footprints v1.2
Parts:
- added C3, C4, C5: 0.1u, Capacitor_SMD:C_1206_3216Metric_Pad1.33x1.80mm_HandSolder, symbol Device:C_Small_US
- added C6, C7, C8, C9: 100u, Capacitor_SMD:CP_Elec_3x5.3, symbol Device:C_Polarized_Small_US
- C1: footprint (none) -> Capacitor_SMD:CP_Elec_3x5.3
- C2: footprint (none) -> Capacitor_SMD:C_1206_3216Metric_Pad1.33x1.80mm_HandSolder
- D1, D10, D11, D2, D3, D4, D5, D9: footprint (none) -> LED_SMD:LED_1206_3216Metric_Pad1.42x1.75mm_HandSolder
- J1: footprint (none) -> Connector_BarrelJack:BarrelJack_CLIFF_FC681465S_SMT_Horizontal
- J2, J3, J4: footprint (none) -> TerminalBlock_Phoenix:TerminalBlock_Phoenix_MKDS-1,5-2-5.08_1x02_P5.08mm_Horizontal
- Q1, Q2, Q3: footprint Package_TO_SOT_THT:TO-220-3_Vertical -> TN0702N3-G:TRANS_TP2104N3-G
- R1, R10, R11, R12, R13, R14, R2, R3, R4, R5, R6, R7, R8, R9: footprint (none) -> Resistor_SMD:R_1206_3216Metric_Pad1.30x1.75mm_HandSolder
- RV1: footprint (none) -> Potentiometer_THT:Potentiometer_Vishay_43_Horizontal
- SW1, SW2: footprint (none) -> Button_Switch_THT:SW_DIP_SPSTx01_Slide_6.7x4.1mm_W7.62mm_P2.54mm_LowProfile
- SW3: footprint (none) -> Button_Switch_THT:SW_PUSH_6mm
Connections:
- net FP_12V: now also C7.1, C8.1, C9.1
- net GND: now also C3.2, C4.2, C5.2, C6.2, C7.2, C8.2, C9.2
- net VDD: now also C3.1, C4.1, C5.1
- net at A1.2 (3V3), RV1.1, U4.3 (Vout+): now also C6.1

Commit message: Updated Footpirnt libraries v1.3
Parts:
- D6, D7, D8: footprint Diode_THT:D_DO-41_SOD81_P10.16mm_Horizontal -> Diode_SMD:D_1206_3216Metric_Pad1.42x1.75mm_HandSolder
Changed lines of the file:
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@@
 			)
 		)
-		(property "Footprint" "Diode_THT:D_DO-41_SOD81_P10.16mm_Horizontal"
+		(property "Footprint" "Diode_SMD:D_1206_3216Metric_Pad1.42x1.75mm_HandSolder"
 			(at 130.175 76.2 0)
 			(effects
@@
 			)
 		)
-		(property "Footprint" "Diode_THT:D_DO-41_SOD81_P10.16mm_Horizontal"
+		(property "Footprint" "Diode_SMD:D_1206_3216Metric_Pad1.42x1.75mm_HandSolder"
 			(at 130.175 142.24 0)
 			(effects
@@
 			)
 		)
-		(property "Footprint" "Diode_THT:D_DO-41_SOD81_P10.16mm_Horizontal"
+		(property "Footprint" "Diode_SMD:D_1206_3216Metric_Pad1.42x1.75mm_HandSolder"
 			(at 130.175 109.22 0)
 			(effects
