File: KiCad/Integrated_System/integrated_system/ECU.kicad_pcb (KiCad board)
At the start: 2 copper layers, 106.5 x 81 mm, 50 parts, among them J1 Jack-DC, J2 Fan 1, J3 Fan 2, J4 Fan 3, Q1 BSS138, Q2 BSS138, Q3 BSS138, SW1 SW_SPDT, SW2 SW_SPDT, SW3 SW_Push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

Commit message: Rough Board layout
Parts:
- U5: moved to B.Cu
- moved C1 85.2 mm to (193.0, 78.0)
- moved C6 85.2 mm to (193.0, 82.9)
- moved C7 85.2 mm to (193.0, 87.8)
- moved C8 85.2 mm to (193.0, 92.6)
- moved C9 85.2 mm to (193.0, 97.5)
- moved U1 61.0 mm to (191.8, 102.4)
- moved U2 59.2 mm to (187.2, 103.3)
- moved SW1 57.4 mm to (182.7, 126.0)
- moved A1 53.8 mm to (133.5, 83.9)
- moved J4 48.9 mm to (166.0, 69.1)
- moved C2 47.5 mm to (184.7, 88.1)
- moved C4 47.5 mm to (184.7, 94.8)
- moved C3 47.5 mm to (184.7, 91.4)
- moved C5 47.5 mm to (184.7, 98.1)
- moved R10 46.4 mm to (166.8, 94.7)
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Other:
- board size 106.5 x 81 mm -> 78.2 x 69.2 mm
- board text added: "4/22/2026"
- board text added: "OSSEM v1.1"
- board text removed: "4/21/2026"
- board text removed: "OSSEM v1.0"

Commit message: updates
Parts:
- removed U5: SCD30, SCD30:MODULE_SCD30
- added U3: SCD30, SCD30:MODULE_SCD30, B.Cu at (138.8, 108.9)
- moved D1 81.9 mm to (91.0, 93.1)
- moved D2 81.9 mm to (91.0, 96.5)
- moved D3 81.9 mm to (91.0, 99.9)
- moved D4 81.9 mm to (91.0, 103.3)
- moved D5 81.9 mm to (91.0, 106.7)
- moved D6 81.9 mm to (91.0, 110.1)
- moved R10 81.9 mm to (85.0, 99.7)
- moved R11 81.9 mm to (85.0, 103.0)
- moved R12 81.9 mm to (85.0, 106.3)
- moved R13 81.9 mm to (85.0, 109.6)
- moved R14 81.9 mm to (85.0, 112.9)
- moved R8 81.9 mm to (85.0, 93.1)
- moved R9 81.9 mm to (85.0, 96.4)
- moved R1 81.9 mm to (79.0, 93.1)
- moved R2 81.9 mm to (79.0, 96.4)
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Other:
- board size 78.2 x 69.2 mm -> 110.2 x 69.2 mm

Commit message: made changes
Parts:
- moved U4 1.07 mm to (175.8, 67.5)
Changed lines of the file:
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@@
 		)
-	)
-	(footprint "Library:Mini360"
-		(layer "F.Cu")
-		(at 176.8125 67.6125)
-		(property "Reference" "U4"
-			(at 8.5 -5 0)
-			(unlocked yes)
-			(layer "F.SilkS")
-			(effects
-				(font
-					(size 1 1)
-					(thickness 0.1)
-				)
-			)
-		)
-		(property "Value" "Mini360 DC to DC Buck Converter 12V to 3.3V"
-			(at 8.5 -3.5 0)
-			(unlocked yes)
-			(layer "F.Fab")
-			(effects
-				(font
-					(size 1 1)
-					(thickness 0.15)
-				)
-			)
-		)
-		(property "Datasheet" ""
-			(at 0 0 0)
-			(unlocked yes)
-			(layer "F.Fab")
-			(hide yes)
-			(effects
-				(font
-					(size 1 1)
-					(thickness 0.15)
-				)
-			)
-		)
-		(property "Description" ""
-			(at 0 0 0)
-			(unlocked yes)
-			(layer "F.Fab")
-			(hide yes)
-			(effects
-				(font
-					(size 1 1)
-					(thickness 0.15)
-				)
-			)
-		)
-		(sheetname "/")
-		(sheetfile "ECU.kicad_sch")
-		(attr through_hole)
-		(fp_rect
-			(start 0 0)
-			(end 17.6 12)
-			(stroke
-				(width 0.05)
-				(type solid)
-			)
-			(fill no)
-			(layer "F.SilkS")
-		)
-		(fp_text user "OUT-"
-			(at 10.5 11.5 0)
-			(unlocked yes)
-			(layer "F.SilkS")
-			(effects
-				(font
-					(size 1 1)
-					(thickness 0.1)
-				)
-				(justify left bottom)
-			)
-		)
-		(fp_text user "IN-"
-			(at 3 11.5 0)
-			(unlocked yes)
-			(layer "F.SilkS")
-			(effects
-				(font
-					(size 1 1)
-					(thickness 0.1)
-				)
-				(justify left bottom)
-			)
-		)
-		(fp_text user "OUT 3V3"
-			(at 4.5 8 0)
-			(unlocked yes)
-			(layer "F.SilkS")
-			(effects
-				(font
-					(size 1 1)
-					(thickness 0.1)
-				)
-				(justify left bottom)
-			)
-		)
-		(fp_text user "IN+"
-			(at 3 2 0)
-			(unlocked yes)
-			(layer "F.SilkS")
-			(effects
-				(font
-					(size 1 1)
-					(thickness 0.1)
-				)
-				(justify left bottom)
-			)
-		)
-		(fp_text user "OUT+"
-			(at 10.5 2 0)
-			(unlocked yes)
-			(layer "F.SilkS")
-			(effects
-				(font
-					(size 1 1)
-					(thickness 0.1)
-				)
-				(justify left bottom)
-			)
-		)
-		(fp_text user "IN 4V5 - 30V"
-			(at 3 5 0)
-			(unlocked yes)
-			(layer "F.SilkS")
-			(effects
-				(font
-					(size 1 1)
-					(thickness 0.1)
-				)
-				(justify left bottom)
-			)
-		)
-		(fp_text user "${REFERENCE}"
-			(at 8.5 -2 0)
-			(unlocked yes)
-			(layer "F.Fab")
-			(effects
-				(font
-					(size 1 1)
-					(thickness 0.15)
-				)
-			)
-		)
-		(pad "1" thru_hole circle
-			(at 1.5 1.5)
-			(size 2.54 2.54)
-			(drill 1.5)
-			(layers "*.Cu" "*.Mask")
-			(remove_unused_layers no)
-			(net 30 "FP_12V")
-			(pinfunction "Vin+")
-			(pintype "input")
-		)
-		(pad "2" thru_hole circle
-			(at 1.5 10.5)
-			(size 2.54 2.54)
-			(drill 1.5)
-			(layers "*.Cu" "*.Mask")
-			(remove_unused_layers no)
-			(net 20 "GND")
-			(pinfunction "Vin-")
-			(pintype "input")
-		)
-		(pad "3" thru_hole circle
-			(at 16 1.5)
-			(size 2.54 2.54)
-			(drill 1.5)
-			(layers "*.Cu" "*.Mask")
-			(remove_unused_layers no)
-			(net 16 "Net-(A1-3V3)")
-			(pinfunction "Vout+")
-			(pintype "output")
-		)
-		(pad "4" thru_hole circle
-			(at 16 10.5)
-			(size 2.54 2.54)
-			(drill 1.5)
-			(layers "*.Cu" "*.Mask")
-			(remove_unused_layers no)
-			(net 20 "GND")
-			(pinfunction "Vout-")
-			(pintype "output")
-		)
-		(embedded_fonts no)
 	)
 	(footprint "Module:Adafruit_Feather"
@@
 		)
 	)
+	(footprint "Library:Mini360"
+		(layer "F.Cu")
+		(at 175.75 67.5)
+		(property "Reference" "U4"
+			(at 8.5 -5 0)
+			(unlocked yes)
+			(layer "F.SilkS")
+			(effects
+				(font
+					(size 1 1)
+					(thickness 0.1)
+				)
+			)
+		)
+		(property "Value" "Mini360 DC to DC Buck Converter 12V to 3.3V"
+			(at 8.5 -3.5 0)
+			(unlocked yes)
+			(layer "F.Fab")
+			(effects
+				(font
+					(size 1 1)
+					(thickness 0.15)
+				)
+			)
+		)
+		(property "Datasheet" ""
+			(at 0 0 0)
+			(unlocked yes)
+			(layer "F.Fab")
+			(hide yes)
+			(effects
+				(font
+					(size 1 1)
+					(thickness 0.15)
+				)
+			)
+		)
+		(property "Description" ""
+			(at 0 0 0)
+			(unlocked yes)
+			(layer "F.Fab")
+			(hide yes)
+			(effects
+				(font
+					(size 1 1)
+					(thickness 0.15)
+				)
+			)
+		)
+		(sheetname "/")
+		(sheetfile "ECU.kicad_sch")
+		(attr through_hole)
+		(fp_rect
+			(start 0 0)
+			(end 17.6 12)
+			(stroke
+				(width 0.05)
+				(type solid)
+			)
+			(fill no)
+			(layer "F.SilkS")
+		)
+		(fp_text user "IN 4V5 - 30V"
+			(at 3 5 0)
+			(unlocked yes)
+			(layer "F.SilkS")
+			(effects
+				(font
+					(size 1 1)
+					(thickness 0.1)
+				)
+				(justify left bottom)
+			)
+		)
+		(fp_text user "OUT 3V3"
+			(at 4.5 8 0)
+			(unlocked yes)
+			(layer "F.SilkS")
+			(effects
+				(font
+					(size 1 1)
+					(thickness 0.1)
+				)
+				(justify left bottom)
+			)
+		)
+		(fp_text user "IN+"
+			(at 12 2 0)
+			(unlocked yes)
+			(layer "F.SilkS")
+			(effects
+				(font
+					(size 1 1)
+					(thickness 0.1)
+				)
+				(justify left bottom)
+			)
+		)
+		(fp_text user "OUT-"
+			(at 3 11 0)
+			(unlocked yes)
+			(layer "F.SilkS")
+			(effects
+				(font
+					(size 1 1)
+					(thickness 0.1)
+				)
+				(justify left bottom)
+			)
+		)
+		(fp_text user "OUT+"
+			(at 3 2 0)
+			(unlocked yes)
+			(layer "F.SilkS")
+			(effects
+				(font
+					(size 1 1)
+					(thickness 0.1)
+				)
+				(justify left bottom)
+			)
+		)
+		(fp_text user "IN-"
+			(at 12 11 0)
+			(unlocked yes)
+			(layer "F.SilkS")
+			(effects
+				(font
+					(size 1 1)
+					(thickness 0.1)
+				)
+				(justify left bottom)
+			)
+		)
+		(fp_text user "${REFERENCE}"
+			(at 8.5 -2 0)
+			(unlocked yes)
+			(layer "F.Fab")
+			(effects
+				(font
+					(size 1 1)
+					(thickness 0.15)
+				)
+			)
+		)
+		(pad "1" thru_hole circle
+			(at 16 1.5)
+			(size 2.54 2.54)
+			(drill 1.3)
+			(layers "*.Cu" "*.Mask")
+			(remove_unused_layers no)
+			(net 30 "FP_12V")
+			(pinfunction "Vin+")
+			(pintype "input")
+		)
+		(pad "2" thru_hole circle
+			(at 16 10.5)
+			(size 2.54 2.54)
+			(drill 1.3)
+			(layers "*.Cu" "*.Mask")
+			(remove_unused_layers no)
+			(net 20 "GND")
+			(pinfunction "Vin-")
+			(pintype "input")
+		)
+		(pad "3" thru_hole circle
+			(at 1.5 1.5)
+			(size 2.54 2.54)
+			(drill 1.3)
+			(layers "*.Cu" "*.Mask")
+			(remove_unused_layers no)
+			(net 16 "Net-(A1-3V3)")
+			(pinfunction "Vout+")
+			(pintype "output")
+		)
+		(pad "4" thru_hole circle
+			(at 1.5 10.5)
+			(size 2.54 2.54)
+			(drill 1.3)
+			(layers "*.Cu" "*.Mask")
+			(remove_unused_layers no)
+			(net 20 "GND")
+			(pinfunction "Vout-")
+			(pintype "output")
+		)
+		(embedded_fonts no)
+	)
 	(footprint "Button_Switch_THT:SW_DIP_SPSTx01_Slide_6.7x4.1mm_W7.62mm_P2.54mm_LowProfile"

Commit message: SGP30 & BME680 Foot print edit
Made a ton of changes
Parts:
- moved U1 34.3 mm to (208.0, 132.6)
- moved U2 20.5 mm to (207.2, 107.8)

Commit message: Nets Label
Parts:
- moved U1 4.47 mm to (206.0, 136.6)

Commit message: redesign v1.3
Parts:
- removed C7, C8, C9: 100u, Capacitor_SMD:CP_Elec_3x5.3
- added SW4: SW_Push, Button_Switch_THT:SW_PUSH_6mm, F.Cu at (113.2, 74.5)
- C1, C6: footprint Capacitor_SMD:CP_Elec_3x5.3 -> Capacitor_SMD:CP_Elec_6.3x7.7
- D10: value LED -> Yellow_LED
- D11: value LED -> Red_LED
- D9: value LED -> Green_LED
- J1: footprint Connector_BarrelJack:BarrelJack_CLIFF_FC681465S_SMT_Horizontal -> Connector_BarrelJack:BarrelJack_GCT_DCJ200-10-A_Horizontal
- RV1: footprint Potentiometer_THT:Potentiometer_Vishay_43_Horizontal -> Potentiometer_THT:Potentiometer_Bourns_3296W_Vertical
- SW1, SW2: footprint Button_Switch_THT:SW_DIP_SPSTx01_Slide_6.7x4.1mm_W7.62mm_P2.54mm_LowProfile -> switch_DM:switch_dm
- U1, U2: moved to B.Cu
- moved R10 191.7 mm to (275.1, 124.1)
- moved R11 191.7 mm to (275.1, 127.4)
- moved R12 191.7 mm to (275.1, 130.7)
- moved R13 191.7 mm to (275.1, 134.0)
- moved R14 191.7 mm to (275.1, 137.3)
- moved R8 191.7 mm to (275.1, 117.5)
- moved R9 191.7 mm to (275.1, 120.8)
- moved R1 191.7 mm to (269.1, 117.5)
- moved R2 191.7 mm to (269.1, 120.8)
- moved R3 191.7 mm to (269.1, 124.1)
- moved R4 191.7 mm to (269.1, 127.4)
- moved R5 191.7 mm to (269.1, 130.7)
- moved R6 191.7 mm to (269.1, 134.0)
- moved R7 191.7 mm to (269.1, 137.3)
- moved D1 176.2 mm to (260.2, 142.1)
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Connections:
- A1 pad 25: unconnected-(A1-A12/IO13-Pad25) -> Net-(A1-A12/IO13)
- U1 pad 1V8: Net-(A1-3V3) -> (no net)
- U1 pad GND: GND -> (no net)
- U1 pad SCL: Net-(A1-SCL/IO22) -> (no net)
- U1 pad SDA: Net-(A1-SDA/IO23) -> (no net)
- U2 pad 3V3: Net-(A1-3V3) -> (no net)
- U2 pad GND: GND -> (no net)
- U2 pad SCK: Net-(A1-SCL/IO22) -> (no net)
- U2 pad SDI: Net-(A1-SDA/IO23) -> (no net)
Routing:
- net (no net): vias 0 -> 4
Other:
- board size 110.2 x 69.2 mm -> 61.3 x 72.8 mm
- board text added: "OSSEM v1.2"
- board text removed: "OSSEM v1.1"

Commit message: Layout Complete
Parts:
- removed RV1: Pot1_Control, Potentiometer_THT:Potentiometer_Bourns_3296W_Vertical
- moved D4 159.2 mm to (109.8, 100.2), turned to 90 degrees
- moved R4 158.7 mm to (110.5, 125.2), turned to 90 degrees
- moved R5 158.6 mm to (110.5, 131.8), turned to 90 degrees
- moved D5 158.1 mm to (109.8, 107.2), turned to 90 degrees
- moved D9 157.2 mm to (129.8, 70.8), turned to 90 degrees
- moved D10 155.5 mm to (133.8, 70.8), turned to 90 degrees
- moved D11 154.0 mm to (137.8, 70.8), turned to 90 degrees
- moved R13 153.6 mm to (133.0, 75.8), turned to 180 degrees
- moved R14 153.3 mm to (133.0, 79.8), turned to 180 degrees
- moved R12 145.7 mm to (142.8, 69.8), turned to 180 degrees
- moved R10 131.9 mm to (144.0, 109.2), turned to 90 degrees
- moved R11 131.3 mm to (144.0, 120.5), turned to 90 degrees
- moved R6 130.3 mm to (144.0, 97.8), turned to 90 degrees
- moved Q1 129.1 mm to (153.0, 93.8)
- moved R9 128.9 mm to (147.7, 101.2)
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Connections:
- net +12V renamed +12V AC to DC wall adapter
Routing:
- net GND: vias 0 -> 2
- net (no net): vias 4 -> 2
Other:
- board text added: "OFF"
- board text added: "ON"

Commit message: Changed 3d model of esp32
Other:
- board text added: "4/23/2026"
- board text added: "OSSEM v1.3"
- board text removed: "4/22/2026"
- board text removed: "OSSEM v1.2"
Changed lines of the file:
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@@
 			)
 		)
+		(model "${KICAD9_3DMODEL_DIR}/esp32grabcad/2821 Adafruit ESP8266 Feather v2.step"
+			(offset
+				(xyz -1.5 6.3 11.5)
+			)
+			(scale
+				(xyz 1 1 1)
+			)
+			(rotate
+				(xyz -0 -0 90)
+			)
+		)
+		(model "${KICAD9_3DMODEL_DIR}/esp32grabcad/Female Header Pitch 2.54mm 1x16 red.stp"
+			(offset
+				(xyz -75 0 0)
+			)
+			(scale
+				(xyz 1 1 1)
+			)
+			(rotate
+				(xyz -0 -0 90)
+			)
+		)
+		(model "${KICAD9_3DMODEL_DIR}/esp32grabcad/Female Header Pitch 2.54mm 1x12 red.stp"
+			(offset
+				(xyz -34.8 -10 0)
+			)
+			(scale
+				(xyz 1 1 1)
+			)
+			(rotate
+				(xyz -0 -0 90)
+			)
+		)
 	)
 	(footprint "Package_TO_SOT_SMD:SOT-23_Handsoldering"
@@
 		(layer "Edge.Cuts")
 	)
-	(gr_text "4/22/2026"
+	(gr_text "4/23/2026"
 		(at 143.75 139 0)
 		(layer "F.SilkS")
@@
 		)
 	)
-	(gr_text "OSSEM v1.2"
+	(gr_text "OSSEM v1.3"
 		(at 143.75 137.5 0)
 		(layer "F.SilkS")
